File: Seminarski.kicad_pcb (KiCad board)
At the start: 2 copper layers, 72.8 x 108 mm, 34 parts, among them SW1 RESET, SW10 SW_Push, SW11 SW_Push, SW12 SW_Push, SW13 SW_Push, SW14 SW_Push, SW15 SW_Push, SW16 SW_Push, SW17 SW_Push, SW18 SW_Push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

Commit message: Veci display
Parts:
- moved U1 2.97 mm to (141.7, 89.1)
- moved BZ1 1.00 mm to (144.5, 60.6)
Routing:
- net BUZZER: track 31.4 -> 36.5 mm
- net +3.3V: track 222.5 -> 226.2 mm
- net C2: track 123.5 -> 119.9 mm
- net C3: track 93.7 -> 90.4 mm
- net C1: track 137.5 -> 134.4 mm
- net R1: track 107.6 -> 104.6 mm
- net GND: track 178.4 -> 181.4 mm
- net RESET: track 63.8 -> 62.2 mm
- net Net-(U1-PC4): track 51.5 -> 52.9 mm
- net C4: track 92.8 -> 91.5 mm
- net Net-(U1-PC5): track 52.0 -> 53.3 mm
- net C5: track 100.4 -> 101.5 mm
- net R4: track 150.7 -> 151.8 mm
- net R3: track 142.3 -> 143.2 mm
- added copper zone on B.Cu, net GND
- added copper zone on F.Cu, net GND
Other:
- board text added: "SIGNAL"

Commit message: Update
Parts:
- C1: value 500uF -> 100uF
- moved U2 0.06 mm to (173.2, 55.2)
Routing:
- net GND: track 181.4 -> 36.3 mm, vias 4 -> 2
