File: Seminarski.kicad_sch (KiCad schematic)
At the start: 34 parts, among them SW1 RESET, SW10 SW_Push, SW11 SW_Push, SW12 SW_Push, SW13 SW_Push, SW14 SW_Push, SW15 SW_Push, SW16 SW_Push, SW17 SW_Push, SW18 SW_Push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

Commit message: Veci display
Parts:
- BT1: Link (none) -> https://www.tme.eu/hr/details/keys1060/baterije-kutije-i-dr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; MANUFACTURER (none) -> KEYSTONE; ManufacturerPartNumber (none) -> 1060
- C1: value 500uF -> 100uF; Link (none) -> https://www.tme.eu/hr/details/ecea0jka101i/kondenzatori-ele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; MANUFACTURER (none) -> PANASONIC; ManufacturerPartNumber (none) -> ECEA0JKA101I
- C2: Link (none) -> https://www.tme.eu/hr/details/cl31b104kbcnnnc/kondenzatori-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; MANUFACTURER (none) -> SAMSUNG; ManufacturerPartNumber (none) -> CL31B104KBCNNNC
- D1: Link (none) -> https://www.tme.eu/hr/details/mm3z3v3t1g/diode-zener-smd/on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; MANUFACTURER (none) -> ONESEMI; ManufacturerPartNumber (none) -> MM3Z3V3T1G
- D2: Link (none) -> https://www.tme.eu/hr/katalog/led-diode-smd-u-boji_113363/?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; MANUFACTURER (none) -> EVERLIGHT; ManufacturerPartNumber (none) -> ELSH-F71G1-0LPNM-CG1G2
- R1: Link (none) -> https://www.tme.eu/hr/details/smd1206-10k-1%25/otpornici-sm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; MANUFACTURER (none) -> ROYALOHM; ManufacturerPartNumber (none) -> 1206S4F1002T5E
- R2: Link (none) -> https://www.tme.eu/hr/details/smd1206-300r-1%25/otpornici-s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; MANUFACTURER (none) -> ROYALOHM; ManufacturerPartNumber (none) -> 1206S4F3000T5E
- R3: Link (none) -> https://www.tme.eu/hr/details/smd1206-330r/otpornici-smd/ro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; MANUFACTURER (none) -> ROYALOHM; ManufacturerPartNumber (none) -> 1206S4J0331T5E
- R4: Link (none) -> https://www.tme.eu/hr/details/smd1206-100r/otpornici-smd/ro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; MANUFACTURER (none) -> ROYALOHM; ManufacturerPartNumber (none) -> 1206S4J0101T5E

Commit message: Update
Parts:
- BZ1: Link (none) -> https://www.tme.eu/hr/details/cmt-9605-85t/signalizatori-el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; MANUFACTURER (none) -> SAME SKY; ManufacturerPartNumber (none) -> CMT-9605-85T
- SW1: Link (none) -> https://www.tme.eu/hr/details/tss61r/mikroprekidaci-tact/kn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; MANUFACTURER (none) -> KNITTER-SWITCH; ManufacturerPartNumber (none) -> TSS 61 R
- SW10, SW11, SW12, SW13, SW14, SW15, SW16, SW17, SW18, SW19, SW2, SW20, SW21, SW3, SW4, SW5, SW6, SW7, SW8, SW9: Link (none) -> https://www.tme.eu/hr/details/tss62n/mikroprekidaci-tact/kn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; MANUFACTURER (none) -> KNITTER-SWITCH; ManufacturerPartNumber (none) -> TSS 62 N
- SW22: Link (none) -> https://www.tme.eu/hr/details/os102011ma1qn1c/prekidaci-kli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; MANUFACTURER (none) -> C&K; ManufacturerPartNumber (none) -> OS102011MA1QN1C
- U1: Link (none) -> https://www.tme.eu/hr/details/atmega328p-pu/obitelj-avr-8-b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; MANUFACTURER (none) -> Microchip; ManufacturerPartNumber (none) -> ATMEGA328P-PU
- U2: Link (none) -> https://www.tme.eu/hr/details/rea012864lwpp3n0/displeji-ole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; MANUFACTURER Displaymodule -> RAYSTAR OPTRONICS; ManufacturerPartNumber (none) -> REA012864LWPP3N00000
Connections:
- no-connect marks 14 -> 13
Other:
- note added: "Matrix tipkala"
- note added: "Mikrokontroler i I2C sučelje displeja"
- note added: "Napajanje, ON/OFF prekidač i signalizacija"
- note added: "Reset za mikrokontroler"
- note added: "Zvučna signalizacija"
- company: (none) -> TVZ
- title: (none) -> Kalkulator
- moved on the sheet: BT1, BZ1, C1, C2, D1, D2, R1, R2, R3, R4, SW1, SW10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
